Commit message: cbf, chaotic version

File: thor_math/ur10/ur10.urdf (robot description, URDF)
Before this commit: robot ur10, 11 links, 10 joints
Links:
- removed link ee_link
- added link base_link_inertia, mass 4.0; collision mesh filename=/home/galileo/projects/thor_ws/src/thor_core/thor_math/ur10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; visual mesh filename=/home/galileo/projects/thor_ws/src/thor_core/thor_math/ur10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
- added link flange
- added link ft_frame
- link base_link: mass 4.0 -> None; geometry 
- link forearm_link: mass 3.87 -> 4.27
- link shoulder_link: mass 7.778 -> 7.1
- link upper_arm_link: mass 12.93 -> 12.7
- link wrist_1_link: mass 1.96 -> 2.0
- link wrist_2_link: mass 1.96 -> 2.0
- link wrist_3_link: mass 0.202 -> 0.365
Joints:
- removed joint ee_fixed_joint
- removed joint world_joint
- removed joint wrist_3_link-tool0_fixed_joint
- added joint base_joint: type fixed, parent world, child base_link, origin xyz=0 0 0 rpy=0 0 0
- added joint base_link-base_link_inertia: type fixed, parent base_link, child base_link_inertia, origin xyz=0 0 0 rpy=0 0 3.141592653589793
- added joint flange-tool0: type fixed, parent flange, child tool0, origin xyz=0 0 0 rpy=1.5707963267948966 0 1.5707963267948966
- added joint wrist_3-flange: type fixed, parent wrist_3_link, child flange, origin xyz=0 0 0 rpy=0 -1.5707963267948966 -1.5707963267948966
- added joint wrist_3_link-ft_frame: type fixed, parent wrist_3_link, child ft_frame, origin xyz=0 0 0 rpy=3.141592653589793 0 0
- joint base_link-base_fixed_joint: origin xyz=0 0 0 rpy=0 0 -3.141592653589793 -> xyz=0 0 0 rpy=0 0 3.141592653589793
- joint elbow_joint: axis 0 1 0 -> 0 0 1; limit lower=-3.141592653589793 upper=3.141592653589793 effort=150.0 velocity=3.15 -> lower=-3.141592653589793 upper=3.141592653589793 effort=150.0 velocity=3.141592653589793; origin xyz=0.0 -0.1719 0.612 rpy=0.0 0.0 0.0 -> xyz=-0.612 0 0 rpy=0 0 0
- joint shoulder_lift_joint: axis 0 1 0 -> 0 0 1; limit lower=-3.141592653589793 upper=3.141592653589793 effort=330.0 velocity=2.16 -> lower=-6.283185307179586 upper=6.283185307179586 effort=330.0 velocity=2.0943951023931953; origin xyz=0.0 0.220941 0.0 rpy=0.0 1.5707963267948966 0.0 -> xyz=0 0 0 rpy=1.570796327 0 0
- joint shoulder_pan_joint: limit lower=-3.141592653589793 upper=3.141592653589793 effort=330.0 velocity=2.16 -> lower=-6.283185307179586 upper=6.283185307179586 effort=330.0 velocity=2.0943951023931953; origin xyz=0.0 0.0 0.1273 rpy=0.0 0.0 0.0 -> xyz=0 0 0.1273 rpy=0 0 0; parent base_link -> base_link_inertia
- joint wrist_1_joint: axis 0 1 0 -> 0 0 1; limit lower=-3.141592653589793 upper=3.141592653589793 effort=54.0 velocity=3.2 -> lower=-6.283185307179586 upper=6.283185307179586 effort=56.0 velocity=3.141592653589793; origin xyz=0.0 0.0 0.5723 rpy=0.0 1.5707963267948966 0.0 -> xyz=-0.5723 0 0.163941 rpy=0 0 0
- joint wrist_2_joint: limit lower=-3.141592653589793 upper=3.141592653589793 effort=54.0 velocity=3.2 -> lower=-6.283185307179586 upper=6.283185307179586 effort=56.0 velocity=3.141592653589793; origin xyz=0.0 0.1149 0.0 rpy=0.0 0.0 0.0 -> xyz=0 -0.1157 -2.373046667922381e-11 rpy=1.570796327 0 0
- joint wrist_3_joint: axis 0 1 0 -> 0 0 1; limit lower=-3.141592653589793 upper=3.141592653589793 effort=54.0 velocity=3.2 -> lower=-6.283185307179586 upper=6.283185307179586 effort=56.0 velocity=3.141592653589793; origin xyz=0.0 0.0 0.1157 rpy=0.0 0.0 0.0 -> xyz=0 0.0922 -1.891053610911353e-11 rpy=1.570796326589793 3.141592653589793 3.141592653589793
